File: sch_doc/zorjadnik_big_pads/file5D41F71D.sch (KiCad schematic (older format))
At the start: 14 parts, among them J8 Conn_01x08, U3 74HC595, U4 74HC595

Commit message: навел красивостей в схеме
Parts:
- CB1, CB2: symbol Device1:CircuitBreaker_1P -> zorjadnik-rescue:CircuitBreaker_1P-Device1
- J8: value Conn_01x08 -> driver; symbol Connector_Generic1:Conn_01x08 -> zorjadnik-rescue:Conn_01x08-Connector_Generic1
- R14, R15: value R -> 100; symbol Device1:R -> zorjadnik-rescue:R-Device1
- R20, R21, R22: value 300 -> 200; symbol Device1:R -> zorjadnik-rescue:R-Device1
- U3, U4: symbol 74xx1:74HC595 -> zorjadnik-rescue:74HC595-74xx1
Connections:
- net D3: now also R20.2; no longer R20.1
- net at D1.8 (CA_DIG3): now also R20.1; no longer R20.2
- net at CB1.2: now also R14.1; no longer R15.1
- net at CB2.2: now also R15.1; no longer R14.1
Other:
- moved on the sheet: CB1, CB2
Changed lines of the file:
@@
 $EndDescr
-$Comp
-L 74xx1:74HC595 U3
-U 1 1 5D42E9F5
-P 2800 2650
-F 0 "U3" H 2500 3200 50  0000 C CNN
-F 1 "74HC595" H 2500 2000 50  0000 C CNN
-F 2 "Package_SO:SOP-16_4.55x10.3mm_P1.27mm" H 2800 2650 50  0001 C CNN
-F 3 "" H 2800 2650 50  0001 C CNN
-	1    2800 2650
-	1    0    0    -1
-$EndComp
 $Comp
 L zorjadnik-rescue:POT-zorjadnik-rescue RV1
@@
 $EndComp
 $Comp
-L power1:+3.3V #PWR021
+L zorjadnik-rescue:+3.3V-power1 #PWR021
 U 1 1 5D42EA04
 P 2050 1050
@@
 $EndComp
 $Comp
-L power1:+3.3V #PWR023
+L zorjadnik-rescue:+3.3V-power1 #PWR023
 U 1 1 5D42EA17
 P 2800 1500
@@
 $EndComp
 $Comp
-L power1:GND #PWR027
+L zorjadnik-rescue:GND-power1 #PWR027
 U 1 1 5D42EA59
 P 2800 5600
@@
 $EndComp
 $Comp
-L power1:+3.3V #PWR030
+L zorjadnik-rescue:+3.3V-power1 #PWR030
 U 1 1 5D42EA87
 P 1450 2050
@@
 $EndComp
 $Comp
-L power1:GND #PWR031
+L zorjadnik-rescue:GND-power1 #PWR031
 U 1 1 5D42EA8D
 P 1300 3200
@@
 $EndComp
 $Comp
-L power1:GND #PWR032
+L zorjadnik-rescue:GND-power1 #PWR032
 U 1 1 5D42EA9A
 P 2950 1950
@@
 Connection ~ 2800 1550
 $Comp
-L power1:GND #PWR034
+L zorjadnik-rescue:GND-power1 #PWR034
 U 1 1 5D42EAEA
 P 2050 1350
@@
 $EndComp
 $Comp
-L power1:GND #PWR035
+L zorjadnik-rescue:GND-power1 #PWR035
 U 1 1 5D42EAF0
 P 2350 2900
@@
 $EndComp
 $Comp
-L Device1:CircuitBreaker_1P CB1
-U 1 1 5D430003
+L zorjadnik-rescue:CircuitBreaker_1P-Device1 CB2
+U 1 1 5D430D68
 P 2300 1750
-F 0 "CB1" H 2375 1750 50  0000 L CNN
-F 1 "CircuitBreaker_1P" H 2375 1825 50  0000 L CNN
+F 0 "CB2" V 2250 1750 50  0000 L CNN
+F 1 "CircuitBreaker_1P" V 2350 1750 50  0000 L CNN
 F 2 "Button_Switch_THT:SW_PUSH_6mm" H 2300 1750 50  0001 C CNN
 F 3 "" H 2300 1750 50  0001 C CNN
@@
 $EndComp
 $Comp
-L Device1:CircuitBreaker_1P CB2
-U 1 1 5D430D68
-P 2300 1600
-F 0 "CB2" H 2375 1600 50  0000 L CNN
-F 1 "CircuitBreaker_1P" H 2375 1675 50  0000 L CNN
-F 2 "Button_Switch_THT:SW_PUSH_6mm" H 2300 1600 50  0001 C CNN
-F 3 "" H 2300 1600 50  0001 C CNN
-	1    2300 1600
-	0    1    1    0
-$EndComp
-$Comp
-L power1:GND #PWR036
+L zorjadnik-rescue:GND-power1 #PWR036
 U 1 1 5D432F85
 P 2650 1800
@@
 	2150 2450 2400 2450
 $Comp
-L Device1:R R21
+L zorjadnik-rescue:R-Device1 R21
 U 1 1 5D6E0909
 P 4850 2600
-F 0 "R21" V 4643 2600 50  0000 C CNN
-F 1 "300" V 4734 2600 50  0000 C CNN
+F 0 "R21" V 4850 2450 50  0000 C CNN
+F 1 "200" V 4850 2600 50  0000 C CNN
 F 2 "Resistor_SMD:R_0805_2012Metric" V 4780 2600 50  0001 C CNN
 F 3 "~" H 4850 2600 50  0001 C CNN
@@
 $EndComp
 $Comp
-L Device1:R R22
+L zorjadnik-rescue:R-Device1 R22
 U 1 1 5D6EBD26
 P 4850 2500
-F 0 "R22" V 4643 2500 50  0000 C CNN
-F 1 "300" V 4734 2500 50  0000 C CNN
+F 0 "R22" V 4750 2500 50  0000 C CNN
+F 1 "200" V 4850 2500 50  0000 C CNN
 F 2 "Resistor_SMD:R_0805_2012Metric" V 4780 2500 50  0001 C CNN
 F 3 "~" H 4850 2500 50  0001 C CNN
@@
 $EndComp
 $Comp
-L Device1:R R20
+L zorjadnik-rescue:R-Device1 R20
 U 1 1 5D6F1DFE
 P 4850 2700
-F 0 "R20" V 4643 2700 50  0000 C CNN
-F 1 "300" V 4734 2700 50  0000 C CNN
+F 0 "R20" V 4750 2700 50  0000 C CNN
+F 1 "200" V 4850 2700 50  0000 C CNN
 F 2 "Resistor_SMD:R_0805_2012Metric" V 4780 2700 50  0001 C CNN
 F 3 "~" H 4850 2700 50  0001 C CNN
 	1    4850 2700
-	0    1    1    0
+	0    -1   -1   0
 $EndComp
 Wire Wire Line
@@
 	1450 2050 1450 3050
 $Comp
-L 74xx1:74HC595 U4
+L zorjadnik-rescue:74HC595-74xx1 U4
 U 1 1 5D50D654
 P 2800 4900
+AR Path="/5D50D654" Ref="U4"  Part="1"
+AR Path="/5D41F71E/5D50D654" Ref="U4"  Part="1"
 F 0 "U4" H 2500 5450 50  0000 C CNN
 F 1 "74HC595" H 2500 4250 50  0000 C CNN
@@
 	3200 4900 3350 4900
 $Comp
-L power1:+3.3V #PWR0109
+L zorjadnik-rescue:+3.3V-power1 #PWR0109
 U 1 1 5D629A6A
 P 2800 3800
@@
 $EndComp
 $Comp
-L power1:GND #PWR0110
+L zorjadnik-rescue:GND-power1 #PWR0110
 U 1 1 5D629A76
 P 2950 4200
@@
 Connection ~ 2800 3850
 $Comp
-L power1:GND #PWR0111
+L zorjadnik-rescue:GND-power1 #PWR0111
 U 1 1 5D6460F2
 P 2800 3350
@@
 	3250 3150 3250 3550
 $Comp
-L power1:GND #PWR0112
+L zorjadnik-rescue:GND-power1 #PWR0112
 U 1 1 5D657AAB
 P 2350 5200
@@
 Connection ~ 3450 3250
 $Comp
-L Device1:R R14
+L zorjadnik-rescue:R-Device1 R14
 U 1 1 5D66A22A
 P 1850 1600
-F 0 "R14" V 1643 1600 50  0000 C CNN
-F 1 "R" V 1734 1600 50  0000 C CNN
+F 0 "R14" V 1750 1600 50  0000 C CNN
+F 1 "100" V 1850 1600 50  0000 C CNN
 F 2 "Resistor_SMD:R_0805_2012Metric" V 1780 1600 50  0001 C CNN
 F 3 "~" H 1850 1600 50  0001 C CNN
@@
 $EndComp
 $Comp
-L Device1:R R15
+L zorjadnik-rescue:R-Device1 R15
 U 1 1 5D66FFB1
 P 1850 1750
-F 0 "R15" V 1643 1750 50  0000 C CNN
-F 1 "R" V 1734 1750 50  0000 C CNN
+F 0 "R15" V 1950 1750 50  0000 C CNN
+F 1 "100" V 1850 1750 50  0000 C CNN
 F 2 "Resistor_SMD:R_0805_2012Metric" V 1780 1750 50  0001 C CNN
 F 3 "~" H 1850 1750 50  0001 C CNN
@@
 	1300 2650 1300 3200
 $Comp
-L Connector_Generic1:Conn_01x08 J8
+L zorjadnik-rescue:Conn_01x08-Connector_Generic1 J8
 U 1 1 5D546DD5
 P 1000 2650
 F 0 "J8" H 918 3167 50  0000 C CNN
-F 1 "Conn_01x08" H 918 3076 50  0000 C CNN
+F 1 "driver" H 918 3076 50  0000 C CNN
 F 2 "Connector_PinHeader_2.54mm:PinHeader_1x08_P2.54mm_Vertical" H 1000 2650 50  0001 C CNN
 F 3 "~" H 1000 2650 50  0001 C CNN
@@
 Wire Wire Line
 	1200 2450 1350 2450
+$Comp
+L zorjadnik-rescue:CircuitBreaker_1P-Device1 CB1
+U 1 1 5D430003
+P 2300 1600
+F 0 "CB1" V 2250 1600 50  0000 L CNN
+F 1 "CircuitBreaker_1P" V 2350 1600 50  0000 L CNN
+F 2 "Button_Switch_THT:SW_PUSH_6mm" H 2300 1600 50  0001 C CNN
+F 3 "" H 2300 1600 50  0001 C CNN
+	1    2300 1600
+	0    1    1    0
+$EndComp
+$Comp
+L zorjadnik-rescue:74HC595-74xx1 U3
+U 1 1 5D42E9F5
+P 2800 2650
+AR Path="/5D42E9F5" Ref="U3"  Part="1"
+AR Path="/5D41F71E/5D42E9F5" Ref="U3"  Part="1"
+F 0 "U3" H 2500 3200 50  0000 C CNN
+F 1 "74HC595" H 2500 2000 50  0000 C CNN
+F 2 "Package_SO:SOP-16_4.55x10.3mm_P1.27mm" H 2800 2650 50  0001 C CNN
+F 3 "" H 2800 2650 50  0001 C CNN
+	1    2800 2650
+	1    0    0    -1
+$EndComp
 Wire Bus Line
 	5200 2400 5200 3250
